Commit message: update sawyer_robot

File: sawyer_description/urdf/LR_sawyer.urdf.xacro (robot description, xacro)
@@ -1,25 +1,36 @@
 <?xml version="1.0" ?>
-<robot xmlns:xacro="http://www.ros.org/wiki/xacro" name="sawyer">
+<robot name="sawyer" xmlns:xacro="http://www.ros.org/wiki/xacro">
   <xacro:arg name="gazebo" default="false"/>
+  <xacro:arg name="pedestal" default="true"/>
+  <xacro:arg name="static" default="true"/>
   <xacro:arg name="electric_gripper" default="false"/>
   <!-- Sawyer Base URDF -->
   <xacro:include filename="$(find sawyer_description)/urdf/LR_sawyer_base.urdf.xacro">
     <xacro:arg name="gazebo" value="${gazebo}"/>
+    <xacro:arg name="pedestal" value="${pedestal}"/>
   </xacro:include>
+  <xacro:if value="$(arg gazebo)">
+  <xacro:include filename="$(find sawyer_description)/urdf/LR_sawyer_base.gazebo.xacro">
+    <xacro:arg name="static" value="${static}"/>
+    <xacro:arg name="pedestal" value="${pedestal}"/>
+  </xacro:include>
+  </xacro:if>
   <!-- Electric Gripper End Effector -->
   <xacro:if value="$(arg electric_gripper)">
-    <xacro:include filename="$(find sawyer_description)/urdf/sawyer_electric_gripper.urdf.xacro">
-      <xacro:arg name="gazebo" value="${gazebo}"/>
-    </xacro:include>
+  <xacro:include filename="$(find sawyer_description)/urdf/sawyer_electric_gripper.urdf.xacro">
+    <xacro:arg name="gazebo" value="${gazebo}"/>
+  </xacro:include>
   </xacro:if>
-<!-- including f/t model
-<xacro:include filename="$(find force_torque_sensor)/model/ft_sensor_ati.urdf.xacro"/>
-<xacro:ft_sensor_nano17 parent="right_hand" name="ft_sensor" type="nano17">
-<origin xyz="0 0 0.005" rpy="0 0 -1.5707"/>
-</xacro:ft_sensor_nano17> -->
-<!-- including f/t model -->
-<xacro:include filename="$(find force_torque_sensor)/model/ft_sensor_ati.urdf.xacro"/>
-<xacro:ft_sensor_axia80 parent="right_hand" name="ft_sensor" type="axia80">
-<origin xyz="0 0 0.005" rpy="0 0 -1.5707"/>
-</xacro:ft_sensor_axia80>
+  <!-- including f/t model
+  <xacro:include filename="$(find force_torque_sensor)/model/ft_sensor_ati.urdf.xacro"/>
+  <xacro:ft_sensor_nano17 parent="right_hand" name="ft_sensor" type="nano17">
+  <origin xyz="0 0 0.005" rpy="0 0 -1.5707"/>
+  </xacro:ft_sensor_nano17> -->
+  <!-- including f/t model -->
+  <xacro:include filename="$(find force_torque_sensor)/model/ft_sensor_ati.urdf.xacro"/>
+  <xacro:ft_sensor_axia80 parent="right_hand" name="ft_sensor" type="axia80">
+  <origin xyz="0 0 0.005" rpy="0 0 -1.5707"/>
+  </xacro:ft_sensor_axia80>
+  <!-- including kinect camera -->
+  <!-- <xacro:include filename="$(find kinect_LR)/model.sdf.xacro"/> -->
 </robot>

File: sawyer_description/urdf/LR_sawyer_base.gazebo.xacro (robot description, xacro)
@@ -1,4 +1,6 @@
 <?xml version="1.0" ?>
 <robot name="baxter" xmlns:xacro="http://www.ros.org/wiki/xacro">
+  <xacro:arg name="pedestal" default="true"/>
+  <xacro:arg name="static" default="true"/>
   <!-- ros_control plugin -->
   <gazebo>
@@ -11,12 +13,16 @@
   </gazebo>
   <!-- Gazebo-Specific Link Properties -->
+<xacro:if value="$(arg static)">
   <link name="world"/>
-    <joint name="fixed" type="fixed">
+  <joint name="fixed" type="fixed">
       <parent link="world"/>
       <child link="base"/>
   </joint>
+</xacro:if>
+<xacro:if value="$(arg pedestal)">
   <gazebo reference="pedestal">
     <material>Gazebo/FlatBlack</material>
   </gazebo>
+</xacro:if>
   <gazebo reference="torso">
     <self_collide>true</self_collide>
@@ -250,135 +256,78 @@
   </transmission>
 <!-- START RAMOS -->
-<!-- commands to start simulation (inc. MoveIt) -->
-<!-- make sure ./intera.sh sim is running -->
-<!-- roslaunch sawyer_gazebo sawyer_world.launch -->
-<!-- rosrun intera_interface enable_robot.py -e -->
-<!-- rosrun intera_interface joint_trajectory_action_server.py -->
-<!-- roslaunch sawyer_moveit_config sawyer_moveit.launch -->
 <!-- DEPTH CAM KINECT_LR -->
 <!-- http://gazebosim.org/tutorials?tut=ros_depth_camera&cat=connect_ros -->
 <!-- rosrun rviz rviz  -->
-<gazebo reference="depth_link">
-  <!-- <sensor type="depth" name="depth1">
-    <plugin name="camera_plugin" filename="libgazebo_ros_openni_kinect.so">
-      <baseline>0.2</baseline>
-      <alwaysOn>true</alwaysOn>
-      <updateRate>0.0</updateRate>
-      <cameraName>kinect</cameraName>
-      <imageTopicName>/kinect/depth/image_raw</imageTopicName>
-      <cameraInfoTopicName>/kinect/depth/camera_info</cameraInfoTopicName>
-      <depthImageTopicName>/kinect/depth/depth_raw</depthImageTopicName>
-      <depthImageInfoTopicName>/kinect/depth/depth_info</depthImageInfoTopicName>
-      <pointCloudTopicName>/kinect/depth/points</pointCloudTopicName>
-      <frameName>depth_link</frameName>
-      <pointCloudCutoff>0.05</pointCloudCutoff>
-      <distortionK1>0</distortionK1>
-      <distortionK2>0</distortionK2>
-      <distortionK3>0</distortionK3>
-      <distortionT1>0</distortionT1>
-      <distortionT2>0</distortionT2>
-      <CxPrime>0</CxPrime>
-      <Cx>0</Cx>
-      <Cy>0</Cy>
-      <focalLength>0</focalLength>
-      <hackBaseline>0</hackBaseline>
-    </plugin> -->
-<!-- from kinect sdf.xacro
-	<plugin name="camera_plugin" filename="libgazebo_ros_openni_kinect.so">
-	  <baseline>0.2</baseline>
-	  <alwaysOn>true</alwaysOn> -->
-	  <!-- Keep this zero, update_rate in the parent <sensor> tag
-	    will control the frame rate.
-	  <updateRate>0.0</updateRate>
-	  <cameraName>camera_kinect</cameraName>
-	  <imageTopicName>/camera_kinect/depth/image_raw</imageTopicName>
-	  <cameraInfoTopicName>/camera_kinect/depth/camera_info</cameraInfoTopicName>
-	  <depthImageTopicName>/camera_kinect/depth/image_raw</depthImageTopicName>
-	  <depthImageInfoTopicName>/camera_kinect/depth/camera_info</depthImageInfoTopicName>
-	  <pointCloudTopicName>/camera_kinect/depth/points</pointCloudTopicName>
-	  <frameName>depth_link</frameName>
-	  <pointCloudCutoff>0.05</pointCloudCutoff>
-	  <distortionK1>0</distortionK1>
-	  <distortionK2>0</distortionK2>
-	  <distortionK3>0</distortionK3>
-	  <distortionT1>0</distortionT1>
-	  <distortionT2>0</distortionT2>
-	  <CxPrime>0</CxPrime>
-	  <Cx>0</Cx>
-	  <Cy>0</Cy>
-	  <focalLength>0</focalLength>
-	  <hackBaseline>0</hackBaseline>
-	</plugin> -->
+  <gazebo reference="depth_link">
 <!-- https://github.com/rosbook/effective_robotics_programming_with_ros/blob/master/chapter7_tutorials/rosbook_arm_description/urdf/sensors/xtion_pro_live.gazebo.xacro -->
-<sensor type="depth" name="depth1_frame_sensor">
-        <always_on>true</always_on>
-        <update_rate>6.0</update_rate>
-        <camera>
-          <!-- <horizontal_fov>1.01229</horizontal_fov>
-          <image>
-            <format>R8G8B8</format>
-            <width>320</width>
-            <height>240</height>
-          </image> -->
-          <clip>
-            <near>0.05</near>
-            <far>4.0</far>
-          </clip>
-        </camera>
-        <plugin name="depth1_frame_controller" filename="libgazebo_ros_openni_kinect.so">
-          <alwaysOn>true</alwaysOn>
-          <updateRate>6.0</updateRate>
-          <cameraName>depth1</cameraName>
-          <imageTopicName>ir/image_raw</imageTopicName>
-          <cameraInfoTopicName>ir/camera_info</cameraInfoTopicName>
-          <depthImageTopicName>depth/image_raw</depthImageTopicName>
-          <depthImageCameraInfoTopicName>depth/camera_info</depthImageCameraInfoTopicName>
-          <pointCloudTopicName>depth/points</pointCloudTopicName>
-          <frameName>depth_link</frameName>
-          <pointCloudCutoff>0.05</pointCloudCutoff>
-          <rangeMax>4.0</rangeMax>
-          <!-- Distortion parameters not supported in gazebo 1.9.* plugins -->
-          <!--distortionK1>0.00000001</distortionK1>
-          <distortionK2>0.00000001</distortionK2>
-          <distortionK3>0.00000001</distortionK3>
-          <distortionT1>0.00000001</distortionT1>
-          <distortionT2>0.00000001</distortionT2-->
-        </plugin>
-      </sensor>
-      <!-- RGB -->
-      <sensor type="depth" name="rgb1_frame_sensor">
-        <always_on>true</always_on>
-        <update_rate>6.0</update_rate>
-        <camera>
-          <!-- <horizontal_fov>1.01229</horizontal_fov>
-          <image>
-            <format>R8G8B8</format>
-            <width>320</width>
-            <height>240</height>
-          </image> -->
-          <clip>
-            <near>0.05</near>
-            <far>4.0</far>
-          </clip>
-        </camera>
-        <plugin name="rgb1_frame_controller" filename="libgazebo_ros_openni_kinect.so">
-          <alwaysOn>true</alwaysOn>
-          <updateRate>6.0</updateRate>
-          <cameraName>rgb1</cameraName>
-          <imageTopicName>rgb/image_raw</imageTopicName>
-          <cameraInfoTopicName>rgb/camera_info</cameraInfoTopicName>
-          <pointCloudTopicName>rgb/points</pointCloudTopicName>
-          <frameName>rbg_link</frameName>
-          <pointCloudCutoff>0.05</pointCloudCutoff>
-          <rangeMax>4.0</rangeMax>
-          <!-- Distortion parameters not supported in gazebo 1.9.* plugins -->
-          <!--distortionK1>0.00000001</distortionK1>
-          <distortionK2>0.00000001</distortionK2>
-          <distortionK3>0.00000001</distortionK3>
-          <distortionT1>0.00000001</distortionT1>
-          <distortionT2>0.00000001</distortionT2-->
-</plugin>
-  </sensor>
-</gazebo>
+    <sensor type="depth" name="depth1_frame_sensor">
+      <update_rate>6.0</update_rate>
+      <camera>
+        <!-- <horizontal_fov>1.01229</horizontal_fov>
+        <image>
+          <format>R8G8B8</format>
+          <width>320</width>
+          <height>240</height>
+        </image> -->
+        <clip>
+          <near>0.05</near>
+          <far>4.0</far>
+        </clip>
+      </camera>
+      <plugin name="depth1_frame_controller" filename="libgazebo_ros_openni_kinect.so">
+        <alwaysOn>true</alwaysOn>
+        <updateRate>6.0</updateRate>
+        <cameraName>depth1</cameraName>
+        <imageTopicName>ir/image_raw</imageTopicName>
+        <cameraInfoTopicName>ir/camera_info</cameraInfoTopicName>
+        <depthImageTopicName>depth/image_raw</depthImageTopicName>
+        <depthImageCameraInfoTopicName>depth/camera_info</depthImageCameraInfoTopicName>
+        <pointCloudTopicName>depth/points</pointCloudTopicName>
+        <frameName>depth_link</frameName>
+        <pointCloudCutoff>0.05</pointCloudCutoff>
+        <rangeMax>4.0</rangeMax>
+        <!-- Distortion parameters not supported in gazebo 1.9.* plugins -->
+        <!--distortionK1>0.00000001</distortionK1>
+        <distortionK2>0.00000001</distortionK2>
+        <distortionK3>0.00000001</distortionK3>
+        <distortionT1>0.00000001</distortionT1>
+        <distortionT2>0.00000001</distortionT2-->
+      </plugin>
+    </sensor>
+    <!-- RGB -->
+    <sensor type="depth" name="rgb1_frame_sensor">
+      <always_on>true</always_on>
+      <update_rate>6.0</update_rate>
+      <camera>
+        <!-- <horizontal_fov>1.01229</horizontal_fov>
+        <image>
+          <format>R8G8B8</format>
+          <width>320</width>
+          <height>240</height>
+        </image> -->
+        <clip>
+          <near>0.05</near>
+          <far>4.0</far>
+        </clip>
+      </camera>
+      <plugin name="rgb1_frame_controller" filename="libgazebo_ros_openni_kinect.so">
+        <alwaysOn>true</alwaysOn>
+        <updateRate>6.0</updateRate>
+        <cameraName>rgb1</cameraName>
+        <imageTopicName>rgb/image_raw</imageTopicName>
+        <cameraInfoTopicName>rgb/camera_info</cameraInfoTopicName>
+        <pointCloudTopicName>rgb/points</pointCloudTopicName>
+        <frameName>rbg_link</frameName>
+        <pointCloudCutoff>0.05</pointCloudCutoff>
+        <rangeMax>4.0</rangeMax>
+        <!-- Distortion parameters not supported in gazebo 1.9.* plugins -->
+        <!--distortionK1>0.00000001</distortionK1>
+        <distortionK2>0.00000001</distortionK2>
+        <distortionK3>0.00000001</distortionK3>
+        <distortionT1>0.00000001</distortionT1>
+        <distortionT2>0.00000001</distortionT2-->
+      </plugin>
+    </sensor>
+  </gazebo>
 <!-- END RAMOS -->
 </robot>

File: sawyer_description/urdf/LR_sawyer_base.urdf.xacro (robot description, xacro)
@@ -2,21 +2,5 @@
 <robot name="sawyer" xmlns:xacro="http://www.ros.org/wiki/xacro">
   <xacro:arg name="gazebo" default="false"/>
-  <xacro:if value="$(arg gazebo)">
-    <!-- Gazebo Tags -->
-    <xacro:include filename="$(find sawyer_description)/urdf/LR_sawyer_base.gazebo.xacro" />
-  </xacro:if>
-  <!-- camera properties -->
-  <!-- https://github.com/richardw05/mybot_ws/tree/master/src/mybot_description/urdf -->
-  <xacro:property name="cameraSize" value="0.05"/>
-  <xacro:property name="cameraMass" value="0.1"/>
-  <xacro:macro name="gazebo_minimum_inertia">
-  <!--  In Gazebo, links with zero principal moment of inertia (ixx, iyy, izz) could lead to infinite acceleration under any finite torque application.
-      http://gazebosim.org/tutorials/?tut=ros_urdf -->
-    <inertial>
-      <origin rpy="0 0 0" xyz="0 0 0"/>
-      <mass value="0.01"/>
-      <inertia ixx="0.01" ixy="0" ixz="0" iyy="0.01" iyz="0" izz="0.01"/>
-    </inertial>
-  </xacro:macro>
+  <xacro:arg name="pedestal" default="true"/>
   <material name="black">
     <color rgba="0 0 0 1"/>
@@ -34,9 +18,5 @@
     <color rgba="0.75294 0.75294 0.75294 1"/>
   </material>
-  <link name="base">
-<xacro:if value="$(arg gazebo)">
-    <xacro:gazebo_minimum_inertia />
-</xacro:if>
-  </link>
+  <link name="base"/>
   <link name="torso">
     <visual>
@@ -49,7 +29,4 @@
       </material>
     </visual>
-<xacro:if value="$(arg gazebo)">
-    <xacro:gazebo_minimum_inertia />
-</xacro:if>
 <xacro:unless value="$(arg gazebo)">
     <inertial>
@@ -60,4 +37,5 @@
 </xacro:unless>
   </link>
+<xacro:if value="$(arg pedestal)">
   <link name="pedestal">
     <visual>
@@ -87,7 +65,4 @@
       </geometry>
     </collision>
-<xacro:if value="$(arg gazebo)">
-    <xacro:gazebo_minimum_inertia />
-</xacro:if>
   </link>
   <joint name="controller_box_fixed" type="fixed">
@@ -103,7 +78,4 @@
       </geometry>
     </collision>
-<xacro:if value="$(arg gazebo)">
-    <xacro:gazebo_minimum_inertia />
-</xacro:if>
   </link>
   <joint name="pedestal_feet_fixed" type="fixed">
@@ -112,4 +84,15 @@
     <child link="pedestal_feet"/>
   </joint>
+  <joint name="pedestal_fixed" type="fixed">
+    <origin rpy="0 0 0" xyz="0.0 0.0 0.0"/>
+    <parent link="base"/>
+    <child link="pedestal"/>
+  </joint>
+</xacro:if>
+  <joint name="right_arm_mount" type="fixed">
+    <origin rpy="0 0 0" xyz="0.0 0.0 0.0"/>
+    <parent link="base"/>
+    <child link="right_arm_base_link"/>
+  </joint>
   <joint name="torso_t0" type="fixed">
     <origin rpy="0 0 0" xyz="0 0 0"/>
@@ -117,14 +100,4 @@
     <child link="torso"/>
   </joint>
-  <joint name="pedestal_fixed" type="fixed">
-    <origin rpy="0 0 0" xyz="0.0 0.0 0.0"/>
-    <parent link="base"/>
-    <child link="pedestal"/>
-  </joint>
-  <joint name="right_arm_mount" type="fixed">
-    <origin rpy="0 0 0" xyz="0.0 0.0 0.0"/>
-    <parent link="base"/>
-    <child link="right_arm_base_link"/>
-  </joint>
   <link name="right_arm_base_link">
     <inertial>
@@ -174,5 +147,5 @@
     <limit effort="80.0" lower="-3.0503" upper="3.0503" velocity="1.74"/>
 <xacro:if value="$(arg gazebo)">
-    <dynamics damping="15.0" friction="5.0"/>
+    <dynamics damping="10.0" friction="5.0"/>
 </xacro:if>
   </joint>
@@ -208,7 +181,4 @@
   </joint>
   <link name="right_torso_itb">
-<xacro:if value="$(arg gazebo)">
-    <xacro:gazebo_minimum_inertia />
-</xacro:if>
 <xacro:unless value="$(arg gazebo)">
     <inertial>
@@ -312,5 +282,5 @@
     <limit effort="40.0" lower="-3.0439" upper="3.0439" velocity="1.957"/>
  <xacro:if value="$(arg gazebo)">
-    <dynamics damping="15.0" friction="5.0"/>
+    <dynamics damping="1.0" friction="0.5"/>
 </xacro:if>
   </joint>
@@ -342,11 +312,8 @@
     <limit effort="9.0" lower="-2.9761" upper="2.9761" velocity="3.485"/>
 <xacro:if value="$(arg gazebo)">
-    <dynamics damping="6.0" friction="1.0"/>
+    <dynamics damping="2.0" friction="1.0"/>
 </xacro:if>
   </joint>
   <link name="right_arm_itb">
-<xacro:if value="$(arg gazebo)">
-    <xacro:gazebo_minimum_inertia />
-</xacro:if>
 <xacro:unless value="$(arg gazebo)">
     <inertial>
@@ -390,12 +357,8 @@
     <limit effort="9.0" lower="-2.9761" upper="2.9761" velocity="3.485"/>
 <xacro:if value="$(arg gazebo)">
-    <dynamics damping="5.5" friction="1.2"/>
-</xacro:if>
-  </joint>
-  <link name="right_hand_camera">
-<xacro:if value="$(arg gazebo)">
-    <xacro:gazebo_minimum_inertia />
-</xacro:if>
-  </link>
+    <dynamics damping="1.0" friction="0.5"/>
+</xacro:if>
+  </joint>
+  <link name="right_hand_camera"/>
   <joint name="right_hand_camera" type="fixed">
     <origin rpy="0 1.57079632679 0" xyz="0.039552 -0.033 0.0695"/>
@@ -404,9 +367,5 @@
     <axis xyz="0 0 0"/>
   </joint>
-  <link name="right_wrist">
-<xacro:if value="$(arg gazebo)">
-    <xacro:gazebo_minimum_inertia />
-</xacro:if>
-  </link>
+  <link name="right_wrist"/>
   <joint name="right_wrist" type="fixed">
     <origin rpy="1.57079632679 0 0" xyz="0 0 0.10541"/>
@@ -445,22 +404,20 @@
 </xacro:if>
 <xacro:unless value="$(arg gazebo)">
-    <limit effort="9.0" lower="-3.14" upper="3.14" velocity="4.545"/>
+    <limit effort="9.0" lower="-4.7124" upper="4.7124" velocity="4.545"/>
 </xacro:unless>
   </joint>
   <link name="right_hand">
-    <!--visual>
+    <collision>
       <origin rpy="0 0 0" xyz="0 0 0.02"/>
       <geometry>
-        <cylinder length="0.08" radius="0.03"/>
-      </geometry>
-    </visual-->
-    <!-- collision>
-      <origin rpy="0 0 0" xyz="0 0 0.02"/>
-      <geometry>
         <cylinder length="0.03" radius="0.035"/>
       </geometry>
-    </collision -->
-<xacro:if value="$(arg gazebo)">
-      <xacro:gazebo_minimum_inertia />
+    </collision>
+<xacro:if value="$(arg gazebo)">
+    <inertial>
+      <origin rpy="0 0 0" xyz="0 0.1 0"/>
+      <mass value="0.01"/>
+      <inertia ixx="0.01" ixy="0.01" ixz="0.01" iyy="0.01" iyz="0.01" izz="0.01"/>
+  </inertial>
 </xacro:if>
 <xacro:unless value="$(arg gazebo)">
@@ -479,7 +436,4 @@
   </joint>
   <link name="right_l1_2">
-<xacro:if value="$(arg gazebo)">
-    <xacro:gazebo_minimum_inertia />
-</xacro:if>
 <xacro:unless value="$(arg gazebo)">
     <inertial>
@@ -503,7 +457,4 @@
   </joint>
   <link name="right_l2_2">
-<xacro:if value="$(arg gazebo)">
-    <xacro:gazebo_minimum_inertia />
-</xacro:if>
 <xacro:unless value="$(arg gazebo)">
     <inertial>
@@ -527,7 +478,4 @@
   </joint>
   <link name="right_l4_2">
-<xacro:if value="$(arg gazebo)">
-    <xacro:gazebo_minimum_inertia />
-</xacro:if>
 <xacro:unless value="$(arg gazebo)">
     <inertial>
@@ -564,7 +512,4 @@
       </geometry>
     </collision>
-<xacro:if value="$(arg gazebo)">
-    <xacro:gazebo_minimum_inertia />
-</xacro:if>
 <xacro:unless value="$(arg gazebo)">
     <inertial>
@@ -580,9 +525,5 @@
     <child link="screen"/>
   </joint>
-  <link name="head_camera">
-<xacro:if value="$(arg gazebo)">
-    <xacro:gazebo_minimum_inertia />
-</xacro:if>
-  </link>
+  <link name="head_camera"/>
   <joint name="head_camera" type="fixed">
     <origin rpy="-2.1293 0 -1.57079632679" xyz="0.0228027 0 0.216572"/>
@@ -595,16 +536,16 @@
 <!-- dir://home/lr101095/.gazebo/models/kinect_LR -->
 <!-- http://gazebosim.org/tutorials?tut=ros_depth_camera&cat=connect_ros -->
-<link name="depth_link">
-  <!-- collision>
-    <origin xyz="-0.1 0 0.025" rpy="0 -1.570796327 0"/>
-      <geometry>
-        <mesh filename="/home/lr101095/ros_ws/underlay/src/kinect_LR/meshes/kinect.dae" />
-      </geometry>
-  </collision -->
+<!-- <link name="depth_link">
   <visual name="visual">
     <geometry>
-      <mesh filename="package://polish_sr300/gazebo_models/models/kinect/meshes/kinect.dae"/>
+      <mesh filename="/home/lr101095/ros_ws/underlay/src/kinect_LR/meshes/kinect.dae" />
     </geometry>
   </visual>
+  <collision>
+    <origin xyz="-0.1 0 0.025" rpy="0 -1.570796327 0"/>
+      <geometry>
+        <mesh filename="/home/lr101095/ros_ws/underlay/src/kinect_LR/meshes/kinect.dae" />
+      </geometry>
+  </collision>
   <sensor name="camera_kinect" type="depth">
     <update_rate>20</update_rate>
@@ -622,13 +563,34 @@
     </camera>
   </sensor>
-</link>
-<joint name="depth_joint" type="fixed">
+</link> -->
+<!-- <joint name="depth_joint" type="fixed">
   <axis xyz="0 1 0" />
-    <!-- origin xyz="0 0 0" rpy="0 0 0"/ -->
     <origin xyz="0 0.1 0.025" rpy="0 -1.570796327 -1.570796327"/>
-    <!-- origin xyz="-0.075 0 0.03" rpy="0 -1.55 0" -->
     <parent link="right_hand"/>
     <child link="depth_link"/>
-</joint>
+</joint> -->
+  <link name="depth_link">
+    <!-- <inertial>
+      <origin rpy="0 0 0" xyz="0 0 0"/>
+      <mass value="0.1"/>
+    </inertial> -->
+    <visual name="visual">
+        <geometry>
+          <mesh filename="/home/lr101095/ros_ws/underlay/src/kinect_LR/meshes/kinect.dae" />
+        </geometry>
+      </visual>
+    <!-- <collision>
+      <geometry>
+         <box>
+           <size>0.073000 0.276000 0.072000</size>
+         </box>
+       </geometry>
+    </collision> -->
+  </link>
+  <joint name="depth_joint" type="fixed">
+    <origin xyz="0 0.1 0.025" rpy="0 -1.570796327 -1.570796327"/>
+    <parent link="right_hand"/>
+    <child link="depth_link"/>
+  </joint>
 <!-- buffing pad geometry -->
 <link name="buffer_l1">
